Commit message: Fixed path in xacro

File: visualization/innolab.urdf.xacro (robot description, xacro)
@@ -2,9 +2,9 @@
 <!-- Kinematic model, simplified visual, no collisions -->
 <robot name="innolab" xmlns:xacro="http://www.ros.org/wiki/xacro">
-<xacro:include filename="$(find atlas_config_flw)/visualization/materials.xacro" />
+<xacro:include filename="$(find atlas_config_example)/visualization/materials.xacro" />
   <link name="base_link">
    <visual>
       <geometry>
-        <mesh scale=".001 .001 .001" filename="file://$(find atlas_config_flw)/visualization/innolab.dae"/>
+        <mesh scale=".001 .001 .001" filename="file://$(find atlas_config_example)/visualization/innolab.dae"/>
       </geometry>
       <origin xyz="-12.5 7.9 0"/>
